File: DragonBoard_rev2.0/DragonBoard.brd (EAGLE design)
At the start: 127.6 x 100 mm, 139 parts, among them IC1 EP4CE15E22C8N, IC2 CP2102, IC3 TPD12S016PWR, J2 RAHHD19TR, X1 PN61729-S

Commit message: fixed HDMI signal names in V2.0, fixed missing I2C resistors in V1.0
Connections:
- net HDMI_BN: now also IC1.136, R7.1; no longer IC1.143, R17.1
- net HDMI_BP: now also IC1.137, R4.1; no longer IC1.144, R16.1
- net HDMI_RN: now also IC1.143, R17.1; no longer IC1.136, R7.1
- net HDMI_RP: now also IC1.144, R16.1; no longer IC1.137, R4.1
Routing:
- net HDMI_RP: track 35.2 -> 43.5 mm
- net HDMI_BP: track 43.5 -> 35.2 mm
- net HDMI_RN: track 26.3 -> 34.6 mm
- net HDMI_BN: track 34.6 -> 26.3 mm
Changed lines of the file:
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@@
 <wire x1="110.2" y1="85.9" x2="110.2" y2="80.355" width="0.254" layer="1"/>
 </signal>
-<signal name="HDMI_RP">
+<signal name="HDMI_BP">
 <contactref element="R4" pad="1"/>
 <contactref element="IC1" pad="137"/>
@@
 <wire x1="44.28" y1="51.378" x2="44.28" y2="60.155" width="0.254" layer="1"/>
 </signal>
-<signal name="HDMI_RN">
+<signal name="HDMI_BN">
 <contactref element="R7" pad="1"/>
 <contactref element="IC1" pad="136"/>
@@
 <wire x1="42.28" y1="51.378" x2="42.28" y2="60.695" width="0.254" layer="1"/>
 </signal>
-<signal name="HDMI_BP">
+<signal name="HDMI_RP">
 <contactref element="R16" pad="1"/>
 <contactref element="IC1" pad="144"/>
@@
 <wire x1="40.78" y1="51.378" x2="40.78" y2="63.005" width="0.254" layer="1"/>
 </signal>
-<signal name="HDMI_BN">
+<signal name="HDMI_RN">
 <contactref element="R17" pad="1"/>
 <contactref element="IC1" pad="143"/>
